Commit message: description: add simulation xacro files
Signed-off-by: Jean Laneurit <jean.laneurit@inrae.fr>

File: romea_rgbd_camera_description/urdf/rgbd_infrared_stereo_camera.xacro (robot description, xacro)
@@ -4,20 +4,35 @@
       params="prefix mode name configuration geometry xyz rpy parent_link mesh_visual ros_namespace">
         <xacro:property name="M_PI" value="3.1415926535897931" />
-        <xacro:property name="link_name" value="${prefix}${name}_link"/>
-        <xacro:property name="joint_name" value="${prefix}${name}_joint"/>
-        <xacro:property name="parent_link_name" value="${prefix}${parent_link}"/>
-        <xacro:property name="baseline" value="${geometry['baseline']}" />
-        <xacro:property name="rgb_camera_x_offset" value="${geometry['rgb_camera_x_offset']}" />
-        <xacro:property name="mass" value="${geometry['mass']}" />
-        <xacro:property name="aabb" value="${geometry['aabb']}" />
-        <xacro:property name="aabb_length" value="${geometry['aabb']['length']}" />
-        <xacro:property name="aabb_width" value="${geometry['aabb']['width']}" />
-        <xacro:property name="aabb_height" value="${geometry['aabb']['height']}" />
-        <xacro:property name="aabb_center" value="${geometry['aabb']['center']}" />
+        <xacro:property name="link_name"
+            value="${prefix}${name}_link"/>
+        <xacro:property name="joint_name"
+            value="${prefix}${name}_joint"/>
+        <xacro:property name="parent_link_name"
+            value="${prefix}${parent_link}"/>
+        <xacro:property name="baseline"
+            value="${geometry['baseline']}" />
+        <xacro:property name="rgb_camera_x_offset"
+            value="${geometry['rgb_camera_x_offset']}" />
+        <xacro:property name="mass"
+            value="${geometry['mass']}" />
+        <xacro:property name="aabb"
+            value="${geometry['aabb']}" />
+        <xacro:property name="aabb_length"
+            value="${geometry['aabb']['length']}" />
+        <xacro:property name="aabb_width"
+            value="${geometry['aabb']['width']}" />
+        <xacro:property name="aabb_height"
+            value="${geometry['aabb']['height']}" />
+        <xacro:property name="aabb_center"
+            value="${geometry['aabb']['center']}" />
         <xacro:if value="${mesh_visual == True and 'mesh' in geometry}">
-        <xacro:property name="mesh_xyz" value="${geometry['mesh']['xyz']}" />
-        <xacro:property name="mesh_rpy" value="${geometry['mesh']['rpy']}" />
-        <xacro:property name="mesh_scale" value="${geometry['mesh']['scale']}" />
-        <xacro:property name="mesh_filename" value="${geometry['mesh']['filename']}" />
+            <xacro:property name="mesh_xyz"
+                value="${geometry['mesh']['xyz']}" />
+            <xacro:property name="mesh_rpy"
+                value="${geometry['mesh']['rpy']}" />
+            <xacro:property name="mesh_scale"
+                value="${geometry['mesh']['scale']}" />
+            <xacro:property name="mesh_filename"
+                value="${geometry['mesh']['filename']}" />
         </xacro:if>
         <!-- Camera Center -->
@@ -59,5 +74,5 @@
             </collision>
         </link>
-        <xacro:if value="${mode == 'simulation'}">
+        <xacro:if value="${'simulation' in mode}">
             <!-- declaration of left and right camera are links are not needed in live mode
                  because TF are published by camera ros driver according extrinsic calibration.
@@ -126,66 +141,12 @@
             </joint>
             <link name="${rgb_camera_optical_frame_name}"/>
-            <!-- due to gazebo limitation only left camera and depth images are published
-                 in the referenced frame of rbg camera optical frame with same size -->
-            <xacro:property name="image_width"
-                value="${configuration['depth_camera']['image_width']}" />
-            <xacro:property name="image_height"
-                value="${configuration['depth_camera']['image_height']}" />
-            <xacro:property name="horizontal_fov"
-                value="${configuration['depth_camera']['horizontal_fov']}" />
-            <xacro:property name="frame_rate"
-                value="${configuration['depth_camera']['frame_rate']}" />
-            <gazebo reference="${link_name}">
-                <material>Gazebo/Red</material>
-                <sensor type="depth" name="${prefix}${name}">
-                    <update_rate>${frame_rate}</update_rate>
-                    <camera>
-                        <horizontal_fov>${horizontal_fov}</horizontal_fov>
-                        <image>
-                            <width>${image_width} </width>
-                            <height>${image_height}</height>
-                            <format>R8G8B8</format>
-                        </image>
-                        <clip>
-                            <near>0.01</near>
-                            <far>100</far>
-                        </clip>
-                        <!-- <noise>
-                        <type>gaussian</type>
-                        <mean>0.0</mean>
-                        <stddev>0.007</stddev>
-                        </noise>
-                        <distortion>
-                        <k1>0.0</k1>
-                        <k2>0.0</k2>
-                        <k3>0.0</k3>
-                        <p1>0.0</p1>
-                        <p2>0.0</p2>
-                        <center>0.5 0.5</center>
-                        </distortion> -->
-                    </camera>
-                    <plugin name="driver" filename="libgazebo_ros_camera.so">
-                        <ros>
-                        <namespace>${ros_namespace}</namespace>
-                        <remapping>camera/camera_info:=rgb/camera_info</remapping>
-                        <remapping>camera/image_raw:=rgb/image_raw</remapping>
-                        <remapping>camera/image_raw/compressed:=rgb/image_raw/compressed</remapping>
-                        <remapping>camera/image_raw/compressedDepth:=rgb/image_raw/compressedDepth</remapping>
-                        <remapping>camera/image_raw/theora:=rgb/image_raw/theora</remapping>
-                        <remapping>camera/depth/camera_info:=depth/camera_info</remapping>
-                        <remapping>camera/depth/image_raw:=depth/image_raw</remapping>
-                        <remapping>camera/depth/image_raw/compressed:=depth/image_raw/compressed</remapping>
-                        <remapping>camera/depth/image_raw/compressedDepth:=depth/image_raw/compressedDepth</remapping>
-                        <remapping>camera/depth/image_raw/theora:=depth/image_raw/theora</remapping>
-                        <remapping>camera/points:=point_cloud/points</remapping>
-                        </ros>
-                        <camera_name>camera</camera_name>
-                        <frame_name>${rgb_camera_optical_joint_name}</frame_name>
-                        <hack_baseline>0.07</hack_baseline>
-                        <min_depth>0.001</min_depth>
-                        <max_depth>300.0</max_depth>
-                    </plugin>
-                </sensor>
-            </gazebo>
+            <xacro:include filename="$(find romea_rgbd_camera_description)/urdf/rgbd_infrared_stereo_camera.simulation.xacro" />
+            <xacro:rgbd_camera_sensor_simulation
+                prefix="${prefix}"
+                mode="${mode}"
+                name="${name}"
+                link_name="${link_name}"
+                configuration="${configuration}"
+                ros_namespace="${ros_namespace}"/>
         </xacro:if>
     </xacro:macro>

File: romea_rgbd_camera_description/urdf/rgbd_stereo_camera.xacro (robot description, xacro)
@@ -4,19 +4,33 @@
       params="prefix mode name configuration geometry xyz rpy parent_link mesh_visual ros_namespace">
         <xacro:property name="M_PI" value="3.1415926535897931" />
-        <xacro:property name="link_name" value="${prefix}${name}_link"/>
-        <xacro:property name="joint_name" value="${prefix}${name}_joint"/>
-        <xacro:property name="parent_link_name" value="${prefix}${parent_link}"/>
-        <xacro:property name="baseline" value="${geometry['baseline']}" />
-        <xacro:property name="mass" value="${geometry['mass']}" />
-        <xacro:property name="aabb" value="${geometry['aabb']}" />
-        <xacro:property name="aabb_length" value="${geometry['aabb']['length']}" />
-        <xacro:property name="aabb_width" value="${geometry['aabb']['width']}" />
-        <xacro:property name="aabb_height" value="${geometry['aabb']['height']}" />
-        <xacro:property name="aabb_center" value="${geometry['aabb']['center']}" />
+        <xacro:property name="link_name"
+            value="${prefix}${name}_link"/>
+        <xacro:property name="joint_name"
+            value="${prefix}${name}_joint"/>
+        <xacro:property name="parent_link_name"
+            value="${prefix}${parent_link}"/>
+        <xacro:property name="baseline"
+            value="${geometry['baseline']}" />
+        <xacro:property name="mass"
+            value="${geometry['mass']}" />
+        <xacro:property name="aabb"
+            value="${geometry['aabb']}" />
+        <xacro:property name="aabb_length"
+            value="${geometry['aabb']['length']}" />
+        <xacro:property name="aabb_width"
+            value="${geometry['aabb']['width']}" />
+        <xacro:property name="aabb_height"
+            value="${geometry['aabb']['height']}" />
+        <xacro:property name="aabb_center"
+            value="${geometry['aabb']['center']}" />
         <xacro:if value="${mesh_visual == True and 'mesh' in geometry}">
-        <xacro:property name="mesh_xyz" value="${geometry['mesh']['xyz']}" />
-        <xacro:property name="mesh_rpy" value="${geometry['mesh']['rpy']}" />
-        <xacro:property name="mesh_scale" value="${geometry['mesh']['scale']}" />
-        <xacro:property name="mesh_filename" value="${geometry['mesh']['filename']}" />
+            <xacro:property name="mesh_xyz"
+                value="${geometry['mesh']['xyz']}" />
+            <xacro:property name="mesh_rpy"
+                value="${geometry['mesh']['rpy']}" />
+            <xacro:property name="mesh_scale"
+                value="${geometry['mesh']['scale']}" />
+            <xacro:property name="mesh_filename"
+                value="${geometry['mesh']['filename']}" />
         </xacro:if>
         <!-- Camera Center -->
@@ -58,5 +72,5 @@
             </collision>
         </link>
-        <xacro:if value="${mode == 'simulation'}">
+        <xacro:if value="${'simulation' in mode}">
             <!-- declaration of left and right camera are links are not needed in live mode
                  because TF are published by camera ros driver according extrinsic calibration.
@@ -104,63 +118,12 @@
             </joint>
             <link name="${right_camera_optical_frame_name}"/>
-            <!-- due to gazebo limitation only left camera and depth images are published
-                 in the referenced frame of left camera optical frame -->
-            <xacro:property name="image_width"
-                value="${configuration['image_width']}" />
-            <xacro:property name="image_height"
-                value="${configuration['image_height']}" />
-            <xacro:property name="horizontal_fov"
-                value="${configuration['horizontal_fov']}" />
-            <xacro:property name="frame_rate"
-                value="${configuration['frame_rate']}" />
-            <gazebo reference="${link_name}">
-                <material>Gazebo/Red</material>
-                <sensor type="depth" name="${prefix}${name}">
-                    <update_rate>${frame_rate}</update_rate>
-                    <camera>
-                        <horizontal_fov>${horizontal_fov}</horizontal_fov>
-                        <image>
-                        <width>${image_width} </width>
-                        <height>${image_height}</height>
-                        <format>R8G8B8</format>
-                        </image>
-                        <clip>
-                        <near>0.01</near>
-                        <far>100</far>
-                        </clip>
-                        <!-- <noise>
-                        <type>gaussian</type>
-                        <mean>0.0</mean>
-                        <stddev>0.007</stddev>
-                        </noise>
-                        <distortion>
-                        <k1>0.0</k1>
-                        <k2>0.0</k2>
-                        <k3>0.0</k3>
-                        <p1>0.0</p1>
-                        <p2>0.0</p2>
-                        <center>0.5 0.5</center>
-                        </distortion> -->
-                    </camera>
-                    <plugin name="driver" filename="libgazebo_ros_camera.so">
-                        <ros>
-                        <namespace>${ros_namespace}</namespace>
-                        <remapping>camera/camera_info:=rgb/camera_info</remapping>
-                        <remapping>camera/image_raw:=rgb/image_raw</remapping>
-                        <remapping>camera/image_raw/compressed:=rgb/image_raw/compressed</remapping>
-                        <remapping>camera/image_raw/compressedDepth:=rgb/image_raw/compressedDepth</remapping>
-                        <remapping>camera/image_raw/theora:=rgb/image_raw/theora</remapping>
-                        <remapping>camera/depth/camera_info:=depth/camera_info</remapping>
-                        <remapping>camera/depth/image_raw:=depth/image_raw</remapping>
-                        <remapping>camera/depth/image_raw/compressed:=depth/image_raw/compressed</remapping>
-                        <remapping>camera/depth/image_raw/compressedDepth:=depth/image_raw/compressedDepth</remapping>
-                        <remapping>camera/depth/image_raw/theora:=depth/image_raw/theora</remapping>
-                        <remapping>camera/points:=point_cloud/points</remapping>
-                        </ros>
-                        <camera_name>camera</camera_name>
-                        <frame_name>${left_camera_optical_frame_name}</frame_name>
-                    </plugin>
-                </sensor>
-            </gazebo>
+            <xacro:include filename="$(find romea_rgbd_camera_description)/urdf/rgbd_stereo_camera.simulation.xacro" />
+            <xacro:rgbd_camera_sensor_simulation
+                prefix="${prefix}"
+                mode="${mode}"
+                name="${name}"
+                link_name="${link_name}"
+                configuration="${configuration}"
+                ros_namespace="${ros_namespace}"/>
         </xacro:if>
     </xacro:macro>

File: romea_rgbd_camera_description/urdf/rgbd_tof_camera.xacro (robot description, xacro)
@@ -4,19 +4,33 @@
       params="prefix mode name configuration geometry xyz rpy parent_link mesh_visual ros_namespace">
         <xacro:property name="M_PI" value="3.1415926535897931" />
-        <xacro:property name="link_name" value="${prefix}${name}_link"/>
-        <xacro:property name="joint_name" value="${prefix}${name}_joint"/>
-        <xacro:property name="parent_link_name" value="${prefix}${parent_link}"/>
-        <xacro:property name="rgb_camera_x_offset" value="${geometry['rgb_camera_x_offset']}" />
-        <xacro:property name="mass" value="${geometry['mass']}" />
-        <xacro:property name="aabb" value="${geometry['aabb']}" />
-        <xacro:property name="aabb_length" value="${geometry['aabb']['length']}" />
-        <xacro:property name="aabb_width" value="${geometry['aabb']['width']}" />
-        <xacro:property name="aabb_height" value="${geometry['aabb']['height']}" />
-        <xacro:property name="aabb_center" value="${geometry['aabb']['center']}" />
+        <xacro:property name="link_name"
+          value="${prefix}${name}_link"/>
+        <xacro:property name="joint_name"
+          value="${prefix}${name}_joint"/>
+        <xacro:property name="parent_link_name"
+          value="${prefix}${parent_link}"/>
+        <xacro:property name="rgb_camera_x_offset"
+          value="${geometry['rgb_camera_x_offset']}" />
+        <xacro:property name="mass"
+          value="${geometry['mass']}" />
+        <xacro:property name="aabb"
+          value="${geometry['aabb']}" />
+        <xacro:property name="aabb_length"
+          value="${geometry['aabb']['length']}" />
+        <xacro:property name="aabb_width"
+          value="${geometry['aabb']['width']}" />
+        <xacro:property name="aabb_height"
+          value="${geometry['aabb']['height']}" />
+        <xacro:property name="aabb_center"
+          value="${geometry['aabb']['center']}" />
         <xacro:if value="${mesh_visual == True and 'mesh' in geometry}">
-          <xacro:property name="mesh_xyz" value="${geometry['mesh']['xyz']}" />
-          <xacro:property name="mesh_rpy" value="${geometry['mesh']['rpy']}" />
-          <xacro:property name="mesh_scale" value="${geometry['mesh']['scale']}" />
-          <xacro:property name="mesh_filename" value="${geometry['mesh']['filename']}" />
+          <xacro:property name="mesh_xyz"
+            value="${geometry['mesh']['xyz']}" />
+          <xacro:property name="mesh_rpy"
+            value="${geometry['mesh']['rpy']}" />
+          <xacro:property name="mesh_scale"
+            value="${geometry['mesh']['scale']}" />
+          <xacro:property name="mesh_filename"
+            value="${geometry['mesh']['filename']}" />
         </xacro:if>
         <!-- Camera Center -->
@@ -58,5 +72,5 @@
             </collision>
         </link>
-      <xacro:if value="${mode == 'simulation'}">
+      <xacro:if value="${'simulation' in mode}">
         <!-- declaration of left and right camera are links are not needed in live mode
               because TF are published by camera ros driver according extrinsic calibration.
@@ -104,63 +118,13 @@
         </joint>
         <link name="${depth_camera_optical_frame_name}"/>
-        <!-- due to gazebo limitation only left camera and depth images are published
-          in the referenced frame of rbg camera optical frame with same size -->
-        <xacro:property name="image_width"
-          value="${configuration['depth_camera']['image_width']}" />
-        <xacro:property name="image_height"
-          value="${configuration['depth_camera']['image_height']}" />
-        <xacro:property name="horizontal_fov"
-          value="${configuration['depth_camera']['horizontal_fov']}" />
-        <xacro:property name="frame_rate"
-          value="${configuration['depth_camera']['frame_rate']}" />
-        <gazebo reference="${link_name}">
-            <material>Gazebo/Red</material>
-            <sensor type="depth" name="${prefix}${name}">
-              <update_rate>${frame_rate}</update_rate>
-              <camera>
-                <horizontal_fov>${horizontal_fov}</horizontal_fov>
-                <image>
-                  <width>${image_width} </width>
-                  <height>${image_height}</height>
-                  <format>R8G8B8</format>
-                </image>
-                <clip>
-                  <near>0.01</near>
-                  <far>100</far>
-                </clip>
-                <!-- <noise>
-                  <type>gaussian</type>
-                  <mean>0.0</mean>
-                  <stddev>0.007</stddev>
-                </noise>
-                <distortion>
-                  <k1>0.0</k1>
-                  <k2>0.0</k2>
-                  <k3>0.0</k3>
-                  <p1>0.0</p1>
-                  <p2>0.0</p2>
-                  <center>0.5 0.5</center>
-                </distortion> -->
-              </camera>
-              <plugin name="driver" filename="libgazebo_ros_camera.so">
-                  <ros>
-                    <remapping>camera/camera_info:=rgb/camera_info</remapping>
-                    <remapping>camera/image_raw:=rgb/image_raw</remapping>
-                    <remapping>camera/image_raw/compressed:=rgb/image_raw/compressed</remapping>
-                    <remapping>camera/image_raw/compressedDepth:=rgb/image_raw/compressedDepth</remapping>
-                    <remapping>camera/image_raw/theora:=rgb/image_raw/theora</remapping>
-                    <remapping>camera/depth/camera_info:=depth/camera_info</remapping>
-                    <remapping>camera/depth/image_raw:=depth/image_raw</remapping>
-                    <remapping>camera/depth/image_raw/compressed:=depth/image_raw/compressed</remapping>
-                    <remapping>camera/depth/image_raw/compressedDepth:=depth/image_raw/compressedDepth</remapping>
-                    <remapping>camera/depth/image_raw/theora:=depth/image_raw/theora</remapping>
-                    <remapping>camera/points:=point_cloud/points</remapping>
-                  </ros>
-                  <camera_name>camera</camera_name>
-                  <frame_name>${rgb_camera_optical_frame_name}</frame_name>
-              </plugin>
-            </sensor>
-          </gazebo>
-        </xacro:if>
-      </xacro:macro>
+        <xacro:include filename="$(find romea_rgbd_camera_description)/urdf/rgbd_tof_camera.simulation.xacro" />
+        <xacro:rgbd_camera_sensor_simulation
+            prefix="${prefix}"
+            mode="${mode}"
+            name="${name}"
+            link_name="${link_name}"
+            configuration="${configuration}"
+            ros_namespace="${ros_namespace}"/>
+    </xacro:if>
+  </xacro:macro>
 </robot>
