Commit message: add unit tests
Signed-off-by: Jean Laneurit <jean.laneurit@inrae.fr>

File: romea_rgbd_camera_description/urdf/rgbd_camera.xacro (robot description, xacro)
@@ -97,4 +97,5 @@
         <link name="${depth_camera_optical_frame_name}"/>
         <gazebo reference="${link_name}">
+          <material>Gazebo/Red</material>
           <sensor type="depth" name="${prefix}${name}">
             <update_rate>${frame_rate}</update_rate>

File: romea_rgbd_camera_description/urdf/rgbd_infrared_stereo_camera.xacro (robot description, xacro)
@@ -1,5 +1,5 @@
 <?xml version="1.0"?>
 <robot xmlns:xacro="http://wiki.ros.org/xacro">
-    <xacro:macro name="stereo_camera_sensor"
+    <xacro:macro name="rgbd_camera_sensor"
       params="prefix mode name configuration geometry xyz rpy parent_link mesh_visual ros_namespace">
         <xacro:property name="M_PI" value="3.1415926535897931" />
@@ -101,6 +101,6 @@
             <joint name="${right_infrared_camera_optical_joint_name}" type="fixed">
                 <origin xyz="0 0 0" rpy="-${M_PI/2} 0.0 -${M_PI/2}"/>
-                <parent link="${right_camera_link_name}"/>
-                <child link="${right_camera_optical_frame_name}"/>
+                <parent link="${right_infrared_camera_link_name}"/>
+                <child link="${right_infrared_camera_optical_frame_name}"/>
             </joint>
             <link name="${right_infrared_camera_optical_frame_name}"/>
@@ -137,29 +137,32 @@
                 value="${configuration['depth_camera']['frame_rate']}" />
             <gazebo reference="${link_name}">
+                <material>Gazebo/Red</material>
                 <sensor type="depth" name="${prefix}${name}">
                     <update_rate>${frame_rate}</update_rate>
-                    <horizontal_fov>${horizontal_fov}</horizontal_fov>
-                    <image>
-                    <width>${image_width} </width>
-                    <height>${image_height}</height>
-                    <format>R8G8B8</format>
-                    </image>
-                    <clip>
-                    <near>0.01</near>
-                    <far>100</far>
-                    </clip>
-                    <!-- <noise>
-                    <type>gaussian</type>
-                    <mean>0.0</mean>
-                    <stddev>0.007</stddev>
-                    </noise>
-                    <distortion>
-                    <k1>0.0</k1>
-                    <k2>0.0</k2>
-                    <k3>0.0</k3>
-                    <p1>0.0</p1>
-                    <p2>0.0</p2>
-                    <center>0.5 0.5</center>
-                    </distortion> -->
+                    <camera>
+                        <horizontal_fov>${horizontal_fov}</horizontal_fov>
+                        <image>
+                            <width>${image_width} </width>
+                            <height>${image_height}</height>
+                            <format>R8G8B8</format>
+                        </image>
+                        <clip>
+                            <near>0.01</near>
+                            <far>100</far>
+                        </clip>
+                        <!-- <noise>
+                        <type>gaussian</type>
+                        <mean>0.0</mean>
+                        <stddev>0.007</stddev>
+                        </noise>
+                        <distortion>
+                        <k1>0.0</k1>
+                        <k2>0.0</k2>
+                        <k3>0.0</k3>
+                        <p1>0.0</p1>
+                        <p2>0.0</p2>
+                        <center>0.5 0.5</center>
+                        </distortion> -->
+                    </camera>
                     <plugin name="driver" filename="libgazebo_ros_camera.so">
                         <ros>
@@ -167,10 +170,19 @@
                         <remapping>camera/camera_info:=rgb/camera_info</remapping>
                         <remapping>camera/image_raw:=rgb/image_raw</remapping>
-                        <remapping>camera/camera_info_depth:=depth/camera_info</remapping>
-                        <remapping>camera/image_depth:=depth/image_raw</remapping>
+                        <remapping>camera/image_raw/compressed:=rgb/image_raw/compressed</remapping>
+                        <remapping>camera/image_raw/compressedDepth:=rgb/image_raw/compressedDepth</remapping>
+                        <remapping>camera/image_raw/theora:=rgb/image_raw/theora</remapping>
+                        <remapping>camera/depth/camera_info:=depth/camera_info</remapping>
+                        <remapping>camera/depth/image_raw:=depth/image_raw</remapping>
+                        <remapping>camera/depth/image_raw/compressed:=depth/image_raw/compressed</remapping>
+                        <remapping>camera/depth/image_raw/compressedDepth:=depth/image_raw/compressedDepth</remapping>
+                        <remapping>camera/depth/image_raw/theora:=depth/image_raw/theora</remapping>
                         <remapping>camera/points:=point_cloud/points</remapping>
                         </ros>
                         <camera_name>camera</camera_name>
                         <frame_name>${rgb_camera_optical_joint_name}</frame_name>
+                        <hack_baseline>0.07</hack_baseline>
+                        <min_depth>0.001</min_depth>
+                        <max_depth>300.0</max_depth>
                     </plugin>
                 </sensor>

File: romea_rgbd_camera_description/urdf/rgbd_stereo_camera.xacro (robot description, xacro)
@@ -1,5 +1,5 @@
 <?xml version="1.0"?>
 <robot xmlns:xacro="http://wiki.ros.org/xacro">
-    <xacro:macro name="stereo_camera_sensor"
+    <xacro:macro name="rgbd_camera_sensor"
       params="prefix mode name configuration geometry xyz rpy parent_link mesh_visual ros_namespace">
         <xacro:property name="M_PI" value="3.1415926535897931" />
@@ -115,29 +115,32 @@
                 value="${configuration['frame_rate']}" />
             <gazebo reference="${link_name}">
+                <material>Gazebo/Red</material>
                 <sensor type="depth" name="${prefix}${name}">
                     <update_rate>${frame_rate}</update_rate>
-                    <horizontal_fov>${horizontal_fov}</horizontal_fov>
-                    <image>
-                    <width>${image_width} </width>
-                    <height>${image_height}</height>
-                    <format>R8G8B8</format>
-                    </image>
-                    <clip>
-                    <near>0.01</near>
-                    <far>100</far>
-                    </clip>
-                    <!-- <noise>
-                    <type>gaussian</type>
-                    <mean>0.0</mean>
-                    <stddev>0.007</stddev>
-                    </noise>
-                    <distortion>
-                    <k1>0.0</k1>
-                    <k2>0.0</k2>
-                    <k3>0.0</k3>
-                    <p1>0.0</p1>
-                    <p2>0.0</p2>
-                    <center>0.5 0.5</center>
-                    </distortion> -->
+                    <camera>
+                        <horizontal_fov>${horizontal_fov}</horizontal_fov>
+                        <image>
+                        <width>${image_width} </width>
+                        <height>${image_height}</height>
+                        <format>R8G8B8</format>
+                        </image>
+                        <clip>
+                        <near>0.01</near>
+                        <far>100</far>
+                        </clip>
+                        <!-- <noise>
+                        <type>gaussian</type>
+                        <mean>0.0</mean>
+                        <stddev>0.007</stddev>
+                        </noise>
+                        <distortion>
+                        <k1>0.0</k1>
+                        <k2>0.0</k2>
+                        <k3>0.0</k3>
+                        <p1>0.0</p1>
+                        <p2>0.0</p2>
+                        <center>0.5 0.5</center>
+                        </distortion> -->
+                    </camera>
                     <plugin name="driver" filename="libgazebo_ros_camera.so">
                         <ros>
@@ -145,6 +148,12 @@
                         <remapping>camera/camera_info:=rgb/camera_info</remapping>
                         <remapping>camera/image_raw:=rgb/image_raw</remapping>
-                        <remapping>camera/camera_info_depth:=depth/camera_info</remapping>
-                        <remapping>camera/image_depth:=depth/image_raw</remapping>
+                        <remapping>camera/image_raw/compressed:=rgb/image_raw/compressed</remapping>
+                        <remapping>camera/image_raw/compressedDepth:=rgb/image_raw/compressedDepth</remapping>
+                        <remapping>camera/image_raw/theora:=rgb/image_raw/theora</remapping>
+                        <remapping>camera/depth/camera_info:=depth/camera_info</remapping>
+                        <remapping>camera/depth/image_raw:=depth/image_raw</remapping>
+                        <remapping>camera/depth/image_raw/compressed:=depth/image_raw/compressed</remapping>
+                        <remapping>camera/depth/image_raw/compressedDepth:=depth/image_raw/compressedDepth</remapping>
+                        <remapping>camera/depth/image_raw/theora:=depth/image_raw/theora</remapping>
                         <remapping>camera/points:=point_cloud/points</remapping>
                         </ros>

File: romea_rgbd_camera_description/urdf/rgbd_tof_camera.xacro (robot description, xacro)
@@ -115,38 +115,44 @@
           value="${configuration['depth_camera']['frame_rate']}" />
         <gazebo reference="${link_name}">
+            <material>Gazebo/Red</material>
             <sensor type="depth" name="${prefix}${name}">
               <update_rate>${frame_rate}</update_rate>
-              <horizontal_fov>${horizontal_fov}</horizontal_fov>
-              <image>
-                <width>${image_width} </width>
-                <height>${image_height}</height>
-                <format>R8G8B8</format>
-              </image>
-              <clip>
-                <near>0.01</near>
-                <far>100</far>
-              </clip>
-              <!-- <noise>
-                <type>gaussian</type>
-                <mean>0.0</mean>
-                <stddev>0.007</stddev>
-              </noise>
-              <distortion>
-                <k1>0.0</k1>
-                <k2>0.0</k2>
-                <k3>0.0</k3>
-                <p1>0.0</p1>
-                <p2>0.0</p2>
-                <center>0.5 0.5</center>
-              </distortion> -->
+              <camera>
+                <horizontal_fov>${horizontal_fov}</horizontal_fov>
+                <image>
+                  <width>${image_width} </width>
+                  <height>${image_height}</height>
+                  <format>R8G8B8</format>
+                </image>
+                <clip>
+                  <near>0.01</near>
+                  <far>100</far>
+                </clip>
+                <!-- <noise>
+                  <type>gaussian</type>
+                  <mean>0.0</mean>
+                  <stddev>0.007</stddev>
+                </noise>
+                <distortion>
+                  <k1>0.0</k1>
+                  <k2>0.0</k2>
+                  <k3>0.0</k3>
+                  <p1>0.0</p1>
+                  <p2>0.0</p2>
+                  <center>0.5 0.5</center>
+                </distortion> -->
               </camera>
               <plugin name="driver" filename="libgazebo_ros_camera.so">
                   <ros>
-                    <namespace>${ros_namespace}</namespace>
-                    <namespace>${ros_namespace}</namespace>
                     <remapping>camera/camera_info:=rgb/camera_info</remapping>
                     <remapping>camera/image_raw:=rgb/image_raw</remapping>
-                    <remapping>camera/camera_info_depth:=depth/camera_info</remapping>
-                    <remapping>camera/image_depth:=depth/image_raw</remapping>
+                    <remapping>camera/image_raw/compressed:=rgb/image_raw/compressed</remapping>
+                    <remapping>camera/image_raw/compressedDepth:=rgb/image_raw/compressedDepth</remapping>
+                    <remapping>camera/image_raw/theora:=rgb/image_raw/theora</remapping>
+                    <remapping>camera/depth/camera_info:=depth/camera_info</remapping>
+                    <remapping>camera/depth/image_raw:=depth/image_raw</remapping>
+                    <remapping>camera/depth/image_raw/compressed:=depth/image_raw/compressed</remapping>
+                    <remapping>camera/depth/image_raw/compressedDepth:=depth/image_raw/compressedDepth</remapping>
+                    <remapping>camera/depth/image_raw/theora:=depth/image_raw/theora</remapping>
                     <remapping>camera/points:=point_cloud/points</remapping>
                   </ros>

Commit message: remove collision in URDF

File: romea_rgbd_camera_description/urdf/rgbd_camera.xacro (robot description, xacro)
@@ -63,10 +63,10 @@
                 </xacro:if>
             </visual>
-            <collision>
+            <!-- <collision>
                 <origin xyz="${aabb_center[0]} ${aabb_center[1]} ${aabb_center[2]}" rpy="0 0 0" />
                 <geometry>
                 <box size="${aabb_length} ${aabb_width} ${aabb_height}" />
                 </geometry>
-            </collision>
+            </collision> -->
         </link>
         <!-- RGB Camera -->

File: romea_rgbd_camera_description/urdf/rgbd_infrared_stereo_camera.xacro (robot description, xacro)
@@ -67,10 +67,10 @@
                 </xacro:if>
             </visual>
-            <collision>
+            <!-- <collision>
                 <origin xyz="${aabb_center[0]} ${aabb_center[1]} ${aabb_center[2]}" rpy="0 0 0" />
                 <geometry>
                 <box size="${aabb_length} ${aabb_width} ${aabb_height}" />
                 </geometry>
-            </collision>
+            </collision> -->
         </link>
         <xacro:if value="${'simulation' in mode}">

File: romea_rgbd_camera_description/urdf/rgbd_stereo_camera.xacro (robot description, xacro)
@@ -65,10 +65,10 @@
                 </xacro:if>
             </visual>
-            <collision>
+            <!-- <collision>
                 <origin xyz="${aabb_center[0]} ${aabb_center[1]} ${aabb_center[2]}" rpy="0 0 0" />
                 <geometry>
                 <box size="${aabb_length} ${aabb_width} ${aabb_height}" />
                 </geometry>
-            </collision>
+            </collision> -->
         </link>
         <xacro:if value="${'simulation' in mode}">

File: romea_rgbd_camera_description/urdf/rgbd_tof_camera.xacro (robot description, xacro)
@@ -65,10 +65,10 @@
                 </xacro:if>
             </visual>
-            <collision>
+            <!-- <collision>
                 <origin xyz="${aabb_center[0]} ${aabb_center[1]} ${aabb_center[2]}" rpy="0 0 0" />
                 <geometry>
                 <box size="${aabb_length} ${aabb_width} ${aabb_height}" />
                 </geometry>
-            </collision>
+            </collision> -->
         </link>
       <xacro:if value="${'simulation' in mode}">
